File: stm32g431cbtx dev module/stm32g431cbtx dev module.kicad_sch (KiCad schematic)
At the start: 18 parts, among them SW1 SW_SPST, U1 STM32G431CBTx, U2 SN65HVD230, X322516MLB4SI 16MHz, 9pF

Commit message: commit
Parts:
- added C13: 100nF, symbol Device:C
- added D1: RED, symbol Device:LED
- added D2: ORANGE, symbol Device:LED
- added J1: I2C, symbol Connector:Conn_01x04_Pin
- added J2: SWD, symbol Connector:Conn_01x04_Pin
- added J3: SPI, symbol Connector:Conn_01x06_Pin
- added R1: 10k, symbol Device:R
- added R2, R3: 5k1, symbol Device:R
Connections:
- net +3V3: now also J1.4 (Pin_4), J2.4 (Pin_4), J3.6 (Pin_6), R1.1, R2.2
- net FDCAN1_RX: now also U2.4 (R)
- net FDCAN1_TX: now also U2.1 (D)
- net GND: now also SW1.2 (B), C13.1, D1.1 (K), D2.1 (K), J1.1 (Pin_1), J2.1 (Pin_1), J3.1 (Pin_1)
- net I2C1_SCL: now also J1.3 (Pin_3)
- net I2C1_SDA: now also J1.2 (Pin_2)
- net NRST: now also SW1.1 (A), C13.2, R1.2
- net SPI1_MISO: now also J3.4 (Pin_4)
- net SPI1_MOSI: now also J3.3 (Pin_3)
- net SPI1_SCK: now also J3.5 (Pin_5)
- net SWCLK: now also J2.2 (Pin_2)
- net SWDIO: now also J2.3 (Pin_3)
- net USER_LED: now also R3.2
- net B0 renamed SPI1_CS
- net SPI1_CS: now also J3.2 (Pin_2)
- new net: D1.2 (A), R2.1
- new net: D2.2 (A), R3.1
